File: standalone_pi_loop.kicad_pcb (KiCad board)
At the start: 4 copper layers, 100 x 100 mm, 40 parts, among them J1 Conn_01x10_Pin, J10 Vout, J11 PI input select, J2 Conn_01x10_Pin, J3 V-sense, J4 Conn_01x05, J5 pot+, J6 pot-, J7 Setpoint, J8 Alt out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

Commit message: Created BOM and pos csv's. Added J4 in pos file
Changed lines of the file:
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@@
 			(at 9.6 -2.47 0)
 			(layer "F.SilkS")
-			(hide yes)
 			(effects
 				(font
@@
 		(sheetname "Root")
 		(sheetfile "standalone_pi_loop.kicad_sch")
-		(attr exclude_from_pos_files)
 		(fp_line
 			(start -1.9 -1.78)
